File: NéO.kicad_sch (KiCad schematic)
At the start: 39 parts, among them J1 RC522, J2 BK-A7670G, J3 POWER, J4 Battery holder, J5 PROGRAMMER, J6 LED, J7 FAN2, J9 FAN1, Q1 IRLML6244, Q2 IRLML6244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

Commit message: Mise à jour des SKU des composants.
Parts:
- C2, C4, C6, C8, C9: SKU 3764069 -> 4740617
- U5: value MCP6006T-E/OT -> AD8591ARTZ-REEL7; SKU 3818589 -> 4019865
Changed lines of the file:
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@@
 			)
 		)
-		(property "SKU" "3764069"
+		(property "SKU" "4740617"
 			(at 173.99 109.22 0)
 			(effects
@@
 			)
 		)
-		(property "Value" "MCP6006T-E/OT"
+		(property "Value" "AD8591ARTZ-REEL7"
 			(at 327.66 109.2514 0)
 			(effects
@@
 			)
 		)
-		(property "SKU" "3818589"
+		(property "SKU" "4019865"
 			(at 317.5 113.03 0)
 			(effects
@@
 			)
 		)
-		(property "SKU" "3764069"
+		(property "SKU" "4740617"
 			(at 80.01 113.03 0)
 			(effects
@@
 			)
 		)
-		(property "SKU" "3764069"
+		(property "SKU" "4740617"
 			(at 218.44 53.34 0)
 			(effects
@@
 			)
 		)
-		(property "SKU" "3764069"
+		(property "SKU" "4740617"
 			(at 248.92 53.34 0)
 			(effects
@@
 			)
 		)
-		(property "SKU" "3764069"
+		(property "SKU" "4740617"
 			(at 309.88 99.06 0)
 			(effects
